File: uart_tool.kicad_pcb (KiCad board)
At the start: 2 copper layers, 4.3 x 11.9 mm, 17 parts, among them J1 Conn_01x03_Pin, J3 Conn_02x05_Odd_Even, U1 AMS1117-3.3, U2 CH340N

Commit message: Add files via upload
Parts:
- moved R1 75.0 mm to (185.5, 87.5), turned to 90 degrees
- moved R4 68.6 mm to (176.1, 96.7), turned to -90 degrees
- moved D1 63.5 mm to (187.5, 87.5), turned to 90 degrees
- moved R3 62.8 mm to (177.0, 101.5), turned to 180 degrees
- moved R2 62.4 mm to (177.0, 99.5), turned to 180 degrees
- moved J3 62.4 mm to (164.2, 104.0), turned to 180 degrees
- moved D4 55.8 mm to (169.5, 95.5)
- moved U2 50.3 mm to (183.0, 101.5), turned to 180 degrees
- moved D3 48.6 mm to (169.5, 100.5)
- moved D2 48.5 mm to (169.5, 98.0)
- moved C3 43.4 mm to (177.0, 103.5)
- moved C1 30.5 mm to (188.2, 92.0), turned to 90 degrees
- moved J1 24.7 mm to (177.5, 87.5), turned to 90 degrees
- moved SW1 24.6 mm to (171.0, 90.0)
- moved C2 19.0 mm to (176.5, 92.0), turned to 90 degrees
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Routing:
- net VBUS: track 0.00 -> 42.4 mm
- net /3.3V: track 0.00 -> 41.3 mm
- net /IO_CTRL: track 0.00 -> 29.0 mm
- net /UART_RX: track 0.00 -> 22.4 mm
- net /UART_TX: track 0.00 -> 17.8 mm
- net /SW_PWR: track 0.00 -> 15.4 mm
- net /USB_D-: track 0.00 -> 12.5 mm
- net /USB_D+: track 0.00 -> 11.3 mm
- net Net-(D4-A): track 0.00 -> 6.60 mm
- net Net-(D2-A): track 0.00 -> 6.33 mm
- net GND: track 0.00 -> 6.31 mm, vias 0 -> 2
- net Net-(D3-A): track 0.00 -> 6.13 mm
- net Net-(U2-V3): track 0.00 -> 2.55 mm
- net Net-(D1-A): track 0.00 -> 2.02 mm
- added copper zone on B.Cu, net GND
- added copper zone on F.Cu, net GND
- added copper zone on F.Cu, net VBUS
Other:
- board size 4.3 x 11.9 mm -> 38.5 x 23.5 mm
- board text added: "3.3V"
- board text added: "5V"
- board text added: "CTRL"
- board text added: "GND"
- board text added: "RX"
- board text added: "TX"
